File: ldo_3V3.kicad_sch (KiCad schematic)
At the start: 3 parts, among them U301 XC6220B331MR-G

Commit message: update SPI pins for OLED
Other:
- company: (none) -> Butler Electronics
Changed lines of the file:
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@@
 (kicad_sch (version 20230121) (generator eeschema)
   (paper "A4")
+  (title_block
+    (date "2024-01-01")
+    (rev "A")
+    (company "Butler Electronics")
+    (comment 1 "Joshua Butler, MD, MHI")
+  )
   (junction (at 43.18 40.64) (diameter 0) (color 0 0 0 0)
   )
